File: DetectorV2.2.kicad_pcb (KiCad board)
At the start: 2 copper layers, 63.3 x 33.4 mm, 29 parts, among them J1 Conn_01x02, U1 AD8092ARZ-REEL7

Commit message: mit version 2.2
Parts:
- moved J1 0.33 mm to (123.7, 80.7)
- moved switch 0.05 mm to (120.0, 94.0)
Routing:
- net GND: track 37.1 -> 29.1 mm, vias 8 -> 10
- net VCC: track 83.7 -> 84.9 mm
Other:
- board text added: "*"
- board text added: "K"
Changed lines of the file:
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@@
 	(footprint "footprints:CONN_SJ-2523-SMT-TR_CUD"
 		(layer "F.Cu")
-		(at 123.99 80.8359 180)
+		(at 123.68 80.72 180)
 		(tags "SJ-2523-SMT-TR ")
 		(property "Reference" "J1"
@@
 		(tags "resistor")
 		(property "Reference" "R6"
-			(at -0.02 -1.67 90)
+			(at -0.0975 1.54 90)
 			(layer "F.SilkS")
 			(effects
@@
 	(footprint "footprints:SSSS810701"
 		(layer "F.Cu")
-		(at 119.97 94.026335)
+		(at 119.98 93.976335)
 		(descr "SSSS810701")
 		(tags "Switch")
@@
 			(layer "F.Fab")
 		)
+		(fp_text user "${REFERENCE}"
+			(at -1.05567 1.691 0)
+			(layer "F.Fab")
+			(hide yes)
+			(effects
+				(font
+					(size 1.27 1.27)
+					(thickness 0.254)
+				)
+			)
+		)
 		(pad "" np_thru_hole circle
 			(at -2.25 1.75)
@@
 		(tags "resistor")
 		(property "Reference" "R8"
-			(at -0.20875 -1.67 90)
+			(at -0.05875 1.56 90)
 			(layer "F.SilkS")
 			(effects
@@
 		(tags "resistor")
 		(property "Reference" "R7"
-			(at 0 -1.5 90)
+			(at -0.37 1.48 90)
 			(layer "F.SilkS")
 			(effects
@@
 	)
 	(gr_text "DIY Particle Detector V2.1\nRojin Aksu \nlaudage@uni-bonn.de"
-		(at 76.08 96.29 0)
+		(at 75.7 96.89 0)
 		(layer "F.SilkS")
 		(effects
@@
 		)
 	)
+	(gr_text "*"
+		(at 92.47 77.21 0)
+		(layer "F.SilkS")
+		(effects
+			(font
+				(size 0.8 0.8)
+				(thickness 0.1875)
+			)
+			(justify left bottom)
+		)
+	)
 	(gr_text "Inspired by Oliver Keller"
-		(at 96.54 97.03 0)
+		(at 96.49 96.82 0)
 		(layer "F.SilkS")
 		(effects
@@
 		)
 	)
+	(gr_text "K"
+		(at 75.44 81.37 0)
+		(layer "F.SilkS")
+		(effects
+			(font
+				(size 1 1)
+				(thickness 0.15)
+			)
+			(justify left bottom)
+		)
+	)
 	(segment
 		(start 98.7375 73.975)
@@
 	)
 	(segment
-		(start 82.7688 83.16)
-		(end 82.7688 82.0912)
-		(width 0.2)
-		(layer "F.Cu")
-		(net 3)
-	)
-	(segment
 		(start 110.05 89.52)
 		(end 111.36 90.83)
@@
 	)
 	(segment
-		(start 115.249386 81.41875)
-		(end 118.97 85.139364)
-		(width 0.2)
+		(start 83.8212 80.5712)
+		(end 82.7688 79.5188)
+		(width 0.25)
 		(layer "F.Cu")
 		(net 3)
@@
 	)
 	(segment
-		(start 112.17 81.21125)
-		(end 114.6025 81.21125)
+		(start 117.835992 83.97)
+		(end 118.97 85.104008)
 		(width 0.25)
 		(layer "F.Cu")
@@
 	)
 	(segment
-		(start 93.03 84.02)
-		(end 93.29 84.28)
+		(start 83.8212 80.5712)
+		(end 82.7688 81.6236)
 		(width 0.25)
 		(layer "F.Cu")
@@
 	)
 	(segment
-		(start 82.7688 79.3888)
-		(end 84.12 80.74)
-		(width 0.2)
+		(start 117.34 83.97)
+		(end 117.835992 83.97)
+		(width 0.25)
+		(layer "F.Cu")
+		(net 3)
+	)
+	(segment
+		(start 93.03 84.02)
+		(end 93.29 84.28)
+		(width 0.25)
 		(layer "F.Cu")
 		(net 3)
@@
 	)
 	(segment
+		(start 118.97 85.104008)
+		(end 118.97 85.4854)
+		(width 0.25)
+		(layer "F.Cu")
+		(net 3)
+	)
+	(segment
 		(start 69.1712 79.7188)
 		(end 68.27 80.62)
@@
 	)
 	(segment
-		(start 118.51 85.358608)
-		(end 118.51 85.74)
+		(start 113.54 81.22)
+		(end 112.17875 81.22)
 		(width 0.25)
 		(layer "F.Cu")
@@
 	)
 	(segment
-		(start 82.7688 78.16)
-		(end 82.7688 79.3888)
-		(width 0.2)
+		(start 118.384088 77.53)
+		(end 118.584391 77.329697)
+		(width 0.25)
+		(layer "F.Cu")
+		(net 3)
+	)
+	(segment
+		(start 82.7688 81.6236)
+		(end 82.7688 83.16)
+		(width 0.25)
+		(layer "F.Cu")
+		(net 3)
+	)
+	(segment
+		(start 112.17875 81.22)
+		(end 112.17 81.21125)
+		(width 0.25)
+		(layer "F.Cu")
+		(net 3)
+	)
+	(segment
+		(start 118.51 85.358608)
+		(end 118.51 85.74)
+		(width 0.25)
 		(layer "F.Cu")
 		(net 3)
@@
 	)
 	(segment
-		(start 114.6025 81.21125)
-		(end 114.81 81.41875)
+		(start 116.45 77.53)
+		(end 118.384088 77.53)
 		(width 0.25)
 		(layer "F.Cu")
@@
 	)
 	(segment
-		(start 114.81 81.41875)
-		(end 115.249386 81.41875)
-		(width 0.2)
-		(layer "F.Cu")
-		(net 3)
-	)
-	(segment
-		(start 82.7688 82.0912)
-		(end 84.12 80.74)
-		(width 0.2)
-		(layer "F.Cu")
-		(net 3)
-	)
-	(segment
 		(start 99.3975 89.3925)
 		(end 99.35 89.44)
@@
 	)
 	(segment
-		(start 106.34 86.695)
-		(end 107.545 86.695)
-		(width 0.2)
-		(layer "F.Cu")
-		(net 3)
-	)
-	(segment
-		(start 118.584391 77.644359)
-		(end 114.81 81.41875)
+		(start 82.7688 79.5188)
+		(end 82.7688 78.16)
 		(width 0.25)
 		(layer "F.Cu")
@@
 	)
 	(segment
-		(start 114.81 81.41875)
-		(end 114.81 81.534056)
+		(start 106.34 86.695)
+		(end 107.545 86.695)
 		(width 0.2)
 		(layer "F.Cu")
@@
 	)
 	(via
-		(at 84.12 80.74)
+		(at 113.54 81.22)
 		(size 0.6)
 		(drill 0.3)
@@
 	)
 	(via
-		(at 114.81 81.41875)
+		(at 99.35 89.44)
 		(size 0.6)
 		(drill 0.3)
@@
 	)
 	(via
-		(at 99.35 89.44)
+		(at 107.56 86.68)
 		(size 0.6)
 		(drill 0.3)
@@
 	)
 	(via
-		(at 107.56 86.68)
+		(at 83.8212 80.5712)
+		(size 0.6)
+		(drill 0.3)
+		(layers "F.Cu" "B.Cu")
+		(free yes)
+		(net 3)
+	)
+	(via
+		(at 116.45 77.53)
+		(size 0.6)
+		(drill 0.3)
+		(layers "F.Cu" "B.Cu")
+		(free yes)
+		(net 3)
+	)
+	(via
+		(at 117.34 83.97)
 		(size 0.6)
 		(drill 0.3)
@@
 	)
 	(segment
-		(start 119.97 92.61)
-		(end 119.97 94.026335)
+		(start 118.97 92.27)
+		(end 118.97 90.5146)
 		(width 0.5)
 		(layer "F.Cu")
@@
 	)
 	(segment
-		(start 97.2526 77.19)
-		(end 97.9638 77.19)
+		(start 119.97 92.61)
+		(end 119.97 94.026335)
 		(width 0.5)
 		(layer "F.Cu")
@@
 	)
 	(segment
-		(start 118.97 91.45)
-		(end 119.38 91.86)
+		(start 97.2526 77.19)
+		(end 97.9638 77.19)
 		(width 0.5)
 		(layer "F.Cu")
@@
 	)
 	(segment
-		(start 119.38 91.86)
-		(end 120.05 92.53)
+		(start 118.97 90.5146)
+		(end 118.97 91.61)
 		(width 0.5)
 		(layer "F.Cu")
@@
 	)
 	(segment
+		(start 118.97 91.61)
+		(end 119.97 92.61)
+		(width 0.5)
+		(layer "F.Cu")
+		(net 10)
+	)
+	(segment
 		(start 84.07 90.29)
 		(end 84.07 86.62)
@@
 	)
 	(segment
-		(start 118.97 90.5146)
-		(end 118.97 91.45)
-		(width 0.5)
-		(layer "F.Cu")
-		(net 10)
-	)
-	(segment
 		(start 108.99 88.65)
 		(end 109.04 88.65)
@@
 	)
 	(segment
-		(start 118.4722 92.7678)
-		(end 119.38 91.86)
-		(width 0.5)
-		(layer "F.Cu")
-		(net 10)
-	)
-	(segment
 		(start 108.99 88.65)
 		(end 108.99 84.61)
@@
 		(width 0.5)
 		(layer "F.Cu")
+		(net 10)
+	)
+	(segment
+		(start 118.4722 92.7678)
+		(end 118.97 92.27)
+		(width 0.5)
+		(layer "F.Cu")

Commit message: updated
Parts:
- added C9: 6n8, Capacitor_SMD:C_0805_2012Metric, F.Cu at (109.2, 80.9)
- added R9: 2.2k, Resistor_SMD:R_0805_2012Metric, F.Cu at (114.2, 80.3)
- R8: value 100k -> 10k
- moved R8 6.14 mm to (107.2, 76.8), turned to 0 degrees
- moved C7 2.09 mm to (113.3, 76.7)
- moved C5 1.24 mm to (105.3, 71.4)
- moved R5 1.24 mm to (105.4, 68.4)
Connections:
- C7 pad 1: Net-(U1-OUT2) -> Net-(C7-Pad1)
- R8 pad 1: /output_signal -> Net-(U1-OUT2)
- R8 pad 2: GND -> Net-(C7-Pad1)
Routing:
- net Net-(C7-Pad1): track 0.00 -> 8.49 mm
- net /output_signal: track 20.5 -> 18.2 mm
- net GND: track 29.1 -> 30.7 mm, vias 10 -> 11
- net Net-(U1--IN2): track 19.7 -> 21.0 mm
- net Net-(U1-OUT2): track 32.7 -> 32.1 mm
Other:
- board text added: "DIY Particle Detector V2.2 Rojin Aksu laudage@uni-bonn.de"
- board text removed: "DIY Particle Detector V2.1 Rojin Aksu laudage@uni-bonn.de"

Commit message: updated
Parts:
- removed R8: 10k, Resistor_SMD:R_0805_2012Metric
- C9: value 6n8 -> C
- moved C9 8.26 mm to (101.8, 77.1)
Connections:
- C7 pad 1: Net-(C7-Pad1) -> Net-(U1-OUT2)
- C9 pad 1: Net-(C7-Pad1) -> VCC
Routing:
- net Net-(C7-Pad1): track 8.49 -> 0.00 mm
- net VCC: track 84.9 -> 91.2 mm
- net Net-(U1--IN2): track 21.0 -> 26.2 mm
- net Net-(U1-OUT2): track 32.1 -> 36.5 mm
