File: DetectorV2.3.kicad_sch (KiCad schematic)
At the start: 26 parts, among them J1 Conn_01x02, SW2 SW_SPST, U1 AD8092ARZ-REEL7

Commit message: updated version 2.3
Parts:
- SW2: footprint footprints:SSSS810701 -> footprints:SWITCH_102AGRLC
Changed lines of the file:
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@@
 			)
 		)
-		(property "Footprint" "footprints:SSSS810701"
+		(property "Footprint" "footprints:SWITCH_102AGRLC"
 			(at 88.9 67.31 0)
 			(effects
