File: DetectorV2.3.kicad_pcb (KiCad board)
At the start: 2 copper layers, 63.3 x 33.4 mm, 8 parts

Commit message: updated version 2.3
Parts:
- added C1: 10p, Capacitor_SMD:C_0805_2012Metric, F.Cu at (85.0, 72.5)
- added C2: 10p, Capacitor_SMD:C_0805_2012Metric, F.Cu at (84.9, 75.2)
- added C3: 100n, Capacitor_SMD:C_0805_2012Metric, F.Cu at (82.3, 85.7)
- added C4: 100n, Capacitor_SMD:C_0805_2012Metric, F.Cu at (89.1, 74.2)
- added C5: 10p, Capacitor_SMD:C_0805_2012Metric, F.Cu at (97.4, 75.2)
- added C6: 100n, Capacitor_SMD:C_0805_2012Metric, F.Cu at (90.6, 84.3)
- added C7: 100n, Capacitor_SMD:C_0805_2012Metric, F.Cu at (97.7, 79.2)
- added C8: 47mikro, footprints:PCAP_EEHZ_D_PAN, F.Cu at (109.1, 81.3)
- added C9: 100n, Capacitor_SMD:C_0805_2012Metric, F.Cu at (91.8, 78.7)
- added J1: Conn_01x02, footprints:CONN_SJ-2523-SMT-TR_CUD, F.Cu at (106.0, 70.1)
- added R1: 4.7k, Resistor_SMD:R_0805_2012Metric, F.Cu at (84.5, 85.7)
- added R2: 15k, Resistor_SMD:R_0805_2012Metric, F.Cu at (86.6, 85.6)
- added R3: 15Mega, Resistor_SMD:R_0805_2012Metric, F.Cu at (85.0, 69.6)
- added R4: 1k, Resistor_SMD:R_0805_2012Metric, F.Cu at (93.2, 74.2)
- added R5: 100k, Resistor_SMD:R_0805_2012Metric, F.Cu at (97.5, 72.0)
- added R6: 10k, Resistor_SMD:R_0805_2012Metric, F.Cu at (92.8, 84.2)
- added R7: 10k, Resistor_SMD:R_0805_2012Metric, F.Cu at (94.9, 84.2)
- added R9: 2.2k, Resistor_SMD:R_0805_2012Metric, F.Cu at (100.8, 82.4)
- added SW2: SW_SPST, footprints:SWITCH_102AGRLC, F.Cu at (117.8, 76.6)
- added TP1: -, Connector_PinHeader_1.00mm:PinHeader_1x01_P1.00mm_Vertical, F.Cu at (117.4, 87.0)
- added TP2: +, Connector_PinHeader_1.00mm:PinHeader_1x01_P1.00mm_Vertical, F.Cu at (117.4, 83.1)
- added U1: AD8092ARZ-REEL7, footprints:R_8_ADI, F.Cu at (85.9, 80.5)
- moved REF** 10.9 mm to (114.9, 93.1)
- moved REF** 10.9 mm to (114.9, 68.1)
Routing:
- net VDD: track 0.00 -> 66.1 mm
- net GND: track 0.00 -> 45.9 mm, vias 0 -> 89
- net Net-(U1-OUT2): track 0.00 -> 36.4 mm
- net /input_signal: track 0.00 -> 24.1 mm
- net /output_signal: track 0.00 -> 18.7 mm
- net Net-(U1--IN2): track 0.00 -> 17.9 mm
- net Net-(U1-OUT1): track 0.00 -> 15.5 mm
- net Net-(U1-+IN1): track 0.00 -> 9.65 mm
- net Net-(U1-+IN2): track 0.00 -> 8.69 mm
- net Net-(SW2-A): track 0.00 -> 4.69 mm
- net Net-(C1-Pad2): track 0.00 -> 3.53 mm
- net Net-(C4-Pad2): track 0.00 -> 2.27 mm
- added copper zone on B.Cu, net GND
- added copper zone on F.Cu, net GND
Other:
- board size 63.3 x 33.4 mm -> 52.4 x 33.4 mm
- board text added: "DIY Particle Detector V2.3 Rojin Aksu laudage@uni-bonn.de"
- board text removed: "DIY Particle Detector V2.2 Rojin Aksu laudage@uni-bonn.de"

Commit message: updated
Parts:
- added G***: LOGO, footprints:NetzwerkTeilchenwelt15mm, F.Cu at (105.2, 92.9)
Other:
- board text added: "+"
- board text added: "-"
- board text added: "DIY Particle Detector V2.3 Rojin Aksu - laudage@uni-bonn.de"
- board text removed: "DIY Particle Detector V2.3 Rojin Aksu laudage@uni-bonn.de"
