File: hardware/DetectorV2.3.kicad_pcb (KiCad board)
At the start: 2 copper layers, 52.4 x 33.4 mm, 31 parts, among them J1 Conn_01x02, SW2 SW_SPST, U1 AD8092ARZ-REEL7

Commit message: updated 2.3 version
Parts:
- moved G*** 0.60 mm to (104.8, 93.3)

Commit message: updated
Routing:
- net GND: vias 89 -> 88
Changed lines of the file:
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@@
-	)
-	(via
-		(at 118 88)
-		(size 0.6)
-		(drill 0.3)
-		(layers "F.Cu" "B.Cu")
-		(net 2)
 	)
 	(via
