File: hardware/Version2.4/DetectorV2.4.kicad_sch (KiCad schematic)
At the start: 28 parts, among them J1 Conn_01x02, SW2 SW_SPST, U1 AD8092ARZ-REEL7

Commit message: 2.4
Parts:
- R3: value 15Mega -> 4.7Mega
- R9: value 2.2k -> 1.6k
Changed lines of the file:
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@@
 			)
 		)
-		(property "Value" "15Mega"
+		(property "Value" "4.7Mega"
 			(at 128.27 63.5 90)
 			(effects
@@
 			)
 		)
-		(property "Value" "2.2k"
+		(property "Value" "1.6k"
 			(at 231.14 124.4599 0)
 			(effects
